Commit message: keyframes fuer X02

File: legged_gym/resources/robots/x02/urdf/xo2.urdf (robot description, URDF)
Before this commit: robot X02Lite, 23 links, 22 joints
Links:
- added link keyframe_head_link
- added link keyframe_left_collar_link
- added link keyframe_left_elbow_link
- added link keyframe_left_hip_link
- added link keyframe_left_knee_link
- added link keyframe_left_shoulder_link
- added link keyframe_pelvis_link
- added link keyframe_right_collar_link
- added link keyframe_right_elbow_link
- added link keyframe_right_hip_link
- added link keyframe_right_knee_link
- added link keyframe_right_shoulder_link
- added link keyframe_torso_link
- added link left_foot_front_link
- added link left_foot_hind_link
- added link left_foot_mid_link
- added link right_foot_front_link
- added link right_foot_hind_link
- added link right_foot_mid_link
Joints:
- removed joint L_hip_pitch
- removed joint L_hip_roll
- removed joint R_hip_roll
- added joint L_hip_pitch_joint: type revolute, parent L_hip_roll_Link, child L_hip_pitch_Link, origin xyz=0.092 -0.001 -2.97932823952292E-05 rpy=-1.5707963267949 0 0, axis 0 0 1, limit lower=-0.5235987755982988 upper=2.007128639793479 effort=72 velocity=9.16297857297023
- added joint L_hip_roll_joint: type revolute, parent L_hip_yaw_Link, child L_hip_roll_Link, origin xyz=0 0.09 -0.0474 rpy=3.14159265358979 1.5707963267949 0, axis 0 0 -1, limit lower=-0.2617993877991494 upper=0.7853981633974483 effort=50 velocity=10.471975511965978
- added joint R_hip_roll_joint: type revolute, parent R_hip_yaw_Link, child R_hip_roll_Link, origin xyz=0 -0.09 0 rpy=0 1.5707963267949 0, axis 0 0 -1, limit lower=-0.2617993877991494 upper=0.7853981633974483 effort=50 velocity=10.471975511965978
- added joint keyframe_head_joint: type fixed, parent torso_Link, child keyframe_head_link, origin xyz=0 0 0.45 rpy=0 0 0
- added joint keyframe_left_collar_joint: type fixed, parent L_shoulder_pitch_Link, child keyframe_left_collar_link, origin xyz=0 0 0.02 rpy=0 0 0
- added joint keyframe_left_elbow_joint: type fixed, parent L_elbow_Link, child keyframe_left_elbow_link, origin xyz=0 0 0 rpy=0 0 0
- added joint keyframe_left_hip_joint: type fixed, parent L_hip_roll_Link, child keyframe_left_hip_link, origin xyz=0 0 0 rpy=0 0 0
- added joint keyframe_left_knee_joint: type fixed, parent L_knee_Link, child keyframe_left_knee_link, origin xyz=0 0 0 rpy=0 0 0
- added joint keyframe_left_shoulder_joint: type fixed, parent L_shoulder_roll_Link, child keyframe_left_shoulder_link, origin xyz=0 0 0 rpy=0 0 0
- added joint keyframe_pelvis_joint: type fixed, parent pelvis, child keyframe_pelvis_link, origin xyz=0 0 -0.075 rpy=0 0 0
- added joint keyframe_right_collar_joint: type fixed, parent R_shoulder_pitch_Link, child keyframe_right_collar_link, origin xyz=0 0 0.02 rpy=0 0 0
- added joint keyframe_right_elbow_joint: type fixed, parent R_elbow_Link, child keyframe_right_elbow_link, origin xyz=0 0 0 rpy=0 0 0
- added joint keyframe_right_hip_joint: type fixed, parent R_hip_roll_Link, child keyframe_right_hip_link, origin xyz=0 0 0 rpy=0 0 0
- added joint keyframe_right_knee_joint: type fixed, parent R_knee_Link, child keyframe_right_knee_link, origin xyz=0 0 0 rpy=0 0 0
- added joint keyframe_right_shoulder_joint: type fixed, parent R_shoulder_roll_Link, child keyframe_right_shoulder_link, origin xyz=0 0 0 rpy=0 0 0
- added joint keyframe_torso_joint: type fixed, parent torso_Link, child keyframe_torso_link, origin xyz=0 0 0.2 rpy=0 0 0
- added joint left_foot_front_joint: type fixed, parent L_ankle_pitch_Link, child left_foot_front_link, origin xyz=0.18 0 -0.06 rpy=0 0 0
- added joint left_foot_hind_joint: type fixed, parent L_ankle_pitch_Link, child left_foot_hind_link, origin xyz=-0.09 0 -0.06 rpy=0 0 0
- added joint left_foot_mid_joint: type fixed, parent L_ankle_pitch_Link, child left_foot_mid_link, origin xyz=0.0 0 -0.06 rpy=0 0 0
- added joint right_foot_front_joint: type fixed, parent R_ankle_pitch_Link, child right_foot_front_link, origin xyz=0.18 0 -0.06 rpy=0 0 0
- added joint right_foot_hind_joint: type fixed, parent R_ankle_pitch_Link, child right_foot_hind_link, origin xyz=-0.09 0 -0.06 rpy=0 0 0
- added joint right_foot_mid_joint: type fixed, parent R_ankle_pitch_Link, child right_foot_mid_link, origin xyz=0.0 0 -0.06 rpy=0 0 0

Commit message: Asset Klasse fertig+URDF

File: legged_gym/resources/robots/x02/urdf/xo2.urdf (robot description, URDF)
Before this commit: robot X02Lite, 42 links, 41 joints
Joints:
- removed joint L_ankle_pitch
- removed joint L_elbow
- removed joint L_knee_pitch
- removed joint L_shoulder_pitch
- removed joint L_shoulder_roll
- removed joint L_shoulder_yaw
- removed joint R_ankle_pitch
- removed joint R_elbow
- removed joint R_hip_pitch
- removed joint R_knee_pitch
- removed joint R_shoulder_pitch
- removed joint R_shoulder_roll
- removed joint R_shoulder_yaw
- removed joint torso
- added joint L_ankle_pitch_joint: type revolute, parent L_knee_Link, child L_ankle_pitch_Link, origin xyz=0.35 0 0 rpy=0 0 0, axis 0 0 1, limit lower=-1.3962634015954636 upper=1.0471975511965976 effort=45 velocity=14.660765716752369
- added joint L_elbow_joint: type fixed, parent L_shoulder_yaw_Link, child L_elbow_Link, origin xyz=0 -0.0100000000001793 0.172999999999993 rpy=1.5707963267949 3.1416 1.5707963267949, axis 0 0 1, limit lower=0.0 upper=2.5307274153917776 effort=14 velocity=5.235987755982989
- added joint L_knee_pitch_joint: type revolute, parent L_hip_pitch_Link, child L_knee_Link, origin xyz=0.349999998731943 -2.9793282395241E-05 0 rpy=0 0 0, axis 0 0 1, limit lower=-2.443460952792061 upper=0.08726646259971647 effort=150 velocity=7.3303828583761845
- added joint L_shoulder_pitch_joint: type fixed, parent torso_Link, child L_shoulder_pitch_Link, origin xyz=0 0.136078524596347 0.306812038248655 rpy=0 1.30899693899577 1.5707963267949, axis 0 0 -1, limit lower=-1.5707963267948966 upper=3.141592653589793 effort=18 velocity=5.235987755982989
- added joint L_shoulder_roll_joint: type fixed, parent L_shoulder_pitch_Link, child L_shoulder_roll_Link, origin xyz=0 0 0.0609999999999959 rpy=-1.5707963267949 0.261799387799122 0, axis 0 0 -1, limit lower=0.0 upper=3.141592653589793 effort=14 velocity=5.235987755982989
- added joint L_shoulder_yaw_joint: type fixed, parent L_shoulder_roll_Link, child L_shoulder_yaw_Link, origin xyz=0.112 0 0 rpy=1.57079632679458 0 1.5707963267949, axis 0 0 -1, limit lower=-2.2689280275926285 upper=2.2689280275926285 effort=14 velocity=5.235987755982989
- added joint R_ankle_pitch_joint: type revolute, parent R_knee_Link, child R_ankle_pitch_Link, origin xyz=0.35 0 0 rpy=0 0 0, axis 0 0 -1, limit lower=-1.3962634015954636 upper=1.0471975511965976 effort=45 velocity=14.660765716752369
- added joint R_elbow_joint: type fixed, parent R_shoulder_yaw_Link, child R_elbow_Link, origin xyz=0 0.00999999999896754 0.173000000000008 rpy=1.5707963267949 0 1.5707963267949, axis 0 0 -1, limit lower=0 upper=1.5707963267949 effort=14 velocity=5.235987755982989
- added joint R_hip_pitch_joint: type revolute, parent R_hip_roll_Link, child R_hip_pitch_Link, origin xyz=0.092 -0.00100000000000001 2.97932823952229E-05 rpy=-1.5707963267949 0 0, axis 0 0 -1, limit lower=-0.5235987755982988 upper=2.007128639793479 effort=72 velocity=9.16297857297023
- added joint R_knee_pitch_joint: type revolute, parent R_hip_pitch_Link, child R_knee_Link, origin xyz=0.349999998731943 2.97932823952059E-05 0 rpy=0 0 0, axis 0 0 -1, limit lower=-2.443460952792061 upper=0.08726646259971647 effort=150 velocity=7.3303828583761845
- added joint R_shoulder_pitch_joint: type fixed, parent torso_Link, child R_shoulder_pitch_Link, origin xyz=0 -0.136078524596347 0.306812038248655 rpy=0 1.30899693899578 -1.5707963267949, axis 0 0 1, limit lower=-1.5707963267948966 upper=3.141592653589793 effort=18 velocity=5.235987755982989
- added joint R_shoulder_roll_joint: type fixed, parent R_shoulder_pitch_Link, child R_shoulder_roll_Link, origin xyz=0 0 0.060999999999996 rpy=-1.5707963267949 0.261799387799122 0, axis 0 0 -1, limit lower=-0.0 upper=3.141592653589793 effort=14 velocity=5.235987755982989
- added joint R_shoulder_yaw_joint: type fixed, parent R_shoulder_roll_Link, child R_shoulder_yaw_Link, origin xyz=0.112 0 0 rpy=1.57079632679458 0 1.5707963267949, axis 0 0 1, limit lower=-2.2689280275926285 upper=2.2689280275926285 effort=14 velocity=5.235987755982989
- added joint torso_joint: type fixed, parent pelvis, child torso_Link, origin xyz=0 0 0 rpy=0 0 0, axis 0 0 1, limit lower=-0.785 upper=0.785 effort=50 velocity=10.471975511965978

Commit message: Init_states-Klasse fertig

File: legged_gym/resources/robots/x02/urdf/xo2.urdf (robot description, URDF)
Before this commit: robot X02Lite, 42 links, 41 joints
Joints:
- joint L_elbow_joint: type fixed -> revolute
- joint L_shoulder_pitch_joint: type fixed -> revolute
- joint L_shoulder_roll_joint: type fixed -> revolute
- joint L_shoulder_yaw_joint: type fixed -> revolute
- joint R_elbow_joint: type fixed -> revolute
- joint R_shoulder_pitch_joint: type fixed -> revolute
- joint R_shoulder_roll_joint: type fixed -> revolute
- joint R_shoulder_yaw_joint: type fixed -> revolute
- joint torso_joint: type fixed -> revolute
