Commit message: relative paths for meshes

File: legged_gym/resources/robots/x02/urdf/x02.urdf (robot description, URDF)
Before this commit: robot X02Lite, 42 links, 41 joints
Links:
- link Head_Link: geometry collision mesh filename=../meshes/Head_Link.STL; visual mesh filename=../meshes/Head_Link.STL
- link L_ankle_pitch_Link: geometry collision cylinder length=0.249 radius=0.018; visual mesh filename=../meshes/L_ankle_pitch_Link.STL
- link L_elbow_Link: geometry collision mesh filename=../meshes/L_elbow_Link.STL; visual mesh filename=../meshes/L_elbow_Link.STL
- link L_hip_pitch_Link: geometry collision mesh filename=../meshes/L_hip_pitch_Link.STL; visual mesh filename=../meshes/L_hip_pitch_Link.STL
- link L_hip_roll_Link: geometry collision mesh filename=../meshes/L_hip_roll_Link.STL; visual mesh filename=../meshes/L_hip_roll_Link.STL
- link L_hip_yaw_Link: geometry collision mesh filename=../meshes/L_hip_yaw_Link.STL; visual mesh filename=../meshes/L_hip_yaw_Link.STL
- link L_knee_Link: geometry collision mesh filename=../meshes/L_knee_Link.STL; visual mesh filename=../meshes/L_knee_Link.STL
- link L_shoulder_pitch_Link: geometry collision mesh filename=../meshes/L_shoulder_pitch_Link.STL; visual mesh filename=../meshes/L_shoulder_pitch_Link.STL
- link L_shoulder_roll_Link: geometry collision mesh filename=../meshes/L_shoulder_roll_Link.STL; visual mesh filename=../meshes/L_shoulder_roll_Link.STL
- link L_shoulder_yaw_Link: geometry collision mesh filename=../meshes/L_shoulder_yaw_Link.STL; visual mesh filename=../meshes/L_shoulder_yaw_Link.STL
- link Logo_Link: geometry collision mesh filename=../meshes/Logo_Link.STL; visual mesh filename=../meshes/Logo_Link.STL
- link R_ankle_pitch_Link: geometry collision cylinder length=0.249 radius=0.018; visual mesh filename=../meshes/R_ankle_pitch_Link.STL
- link R_elbow_Link: geometry collision mesh filename=../meshes/R_elbow_Link.STL; visual mesh filename=../meshes/R_elbow_Link.STL
- link R_hip_pitch_Link: geometry collision mesh filename=../meshes/R_hip_pitch_Link.STL; visual mesh filename=../meshes/R_hip_pitch_Link.STL
- link R_hip_roll_Link: geometry collision mesh filename=../meshes/R_hip_roll_Link.STL; visual mesh filename=../meshes/R_hip_roll_Link.STL
- link R_hip_yaw_Link: geometry collision mesh filename=../meshes/R_hip_yaw_Link.STL; visual mesh filename=../meshes/R_hip_yaw_Link.STL
- link R_knee_Link: geometry collision mesh filename=../meshes/R_knee_Link.STL; visual mesh filename=../meshes/R_knee_Link.STL
- link R_shoulder_pitch_Link: geometry collision mesh filename=../meshes/R_shoulder_pitch_Link.STL; visual mesh filename=../meshes/R_shoulder_pitch_Link.STL
- link R_shoulder_roll_Link: geometry collision mesh filename=../meshes/R_shoulder_roll_Link.STL; visual mesh filename=../meshes/R_shoulder_roll_Link.STL
- link R_shoulder_yaw_Link: geometry collision mesh filename=../meshes/R_shoulder_yaw_Link.STL; visual mesh filename=../meshes/R_shoulder_yaw_Link.STL
- link pelvis: geometry collision mesh filename=../meshes/pelvis.STL; visual mesh filename=../meshes/pelvis.STL
- link torso_link: geometry collision mesh filename=../meshes/torso_link.STL; visual mesh filename=../meshes/torso_link.STL

Commit message: mesh änderung

File: legged_gym/resources/robots/x02/urdf/x02.urdf (robot description, URDF)
Before this commit: robot X02Lite, 42 links, 41 joints
Links:
- link L_ankle_pitch_Link: geometry collision cylinder length=0.249 radius=0.018; visual mesh filename=../meshes/L_ankle_pitch_Link_x02.STL
- link R_ankle_pitch_Link: geometry collision cylinder length=0.249 radius=0.018; visual mesh filename=../meshes/R_ankle_pitch_Link_x02.STL

Commit message: GPU Fehler gelöst

File: legged_gym/resources/robots/x02/urdf/x02.urdf (robot description, URDF)
Before this commit: robot X02Lite, 42 links, 41 joints
Links:
- link L_ankle_pitch_Link: geometry collision cylinder length=0.249 radius=0.018; visual mesh filename=../meshes/L_ankle_pitch_Link.STL
- link R_ankle_pitch_Link: geometry collision cylinder length=0.249 radius=0.018; visual mesh filename=../meshes/R_ankle_pitch_Link.STL

Commit message: neuer Mesh sitzt richtig, Auxiliarys noch falsch

File: legged_gym/resources/robots/x02/urdf/x02.urdf (robot description, URDF)
Before this commit: robot X02Lite, 42 links, 41 joints
Links:
- added link auxiliary_left_ankle_roll_link1; visual sphere radius=0.01
- added link auxiliary_left_ankle_roll_link2; visual sphere radius=0.01
- added link auxiliary_left_ankle_roll_link3; visual sphere radius=0.01
- added link auxiliary_left_ankle_roll_link4; visual sphere radius=0.01
- added link auxiliary_right_ankle_roll_link1; visual sphere radius=0.01
- added link auxiliary_right_ankle_roll_link2; visual sphere radius=0.01
- added link auxiliary_right_ankle_roll_link3; visual sphere radius=0.01
- added link auxiliary_right_ankle_roll_link4; visual sphere radius=0.01
- link L_ankle_pitch_Link: mass 0.256 -> 0.556154115746433; geometry collision sphere radius=0.005; collision sphere radius=0.005
- link R_ankle_pitch_Link: mass 0.256 -> 0.556160945494453; geometry collision sphere radius=0.005; collision sphere radius=0.005
Joints:
- added joint auxiliary_left_ankle_roll_joint1: type fixed, parent L_ankle_pitch_Link, child auxiliary_left_ankle_roll_link1, origin xyz=0.035 0.1 0 rpy=0 0 0
- added joint auxiliary_left_ankle_roll_joint2: type fixed, parent L_ankle_pitch_Link, child auxiliary_left_ankle_roll_link2, origin xyz=0.035 -0.1 0 rpy=0 0 0
- added joint auxiliary_left_ankle_roll_joint3: type fixed, parent L_ankle_pitch_Link, child auxiliary_left_ankle_roll_link3, origin xyz=0.2 0 0 rpy=0 0 0
- added joint auxiliary_left_ankle_roll_joint4: type fixed, parent L_ankle_pitch_Link, child auxiliary_left_ankle_roll_link4, origin xyz=-0.15 0 0 rpy=0 0 0
- added joint auxiliary_right_ankle_roll_joint1: type fixed, parent R_ankle_pitch_Link, child auxiliary_right_ankle_roll_link1, origin xyz=0.035 0.1 0 rpy=0 0 0
- added joint auxiliary_right_ankle_roll_joint2: type fixed, parent R_ankle_pitch_Link, child auxiliary_right_ankle_roll_link2, origin xyz=0.035 -0.1 0 rpy=0 0 0
- added joint auxiliary_right_ankle_roll_joint3: type fixed, parent R_ankle_pitch_Link, child auxiliary_right_ankle_roll_link3, origin xyz=0.2 0 0 rpy=0 0 0
- added joint auxiliary_right_ankle_roll_joint4: type fixed, parent R_ankle_pitch_Link, child auxiliary_right_ankle_roll_link4, origin xyz=-0.15 0 0 rpy=0 0 0
- joint L_ankle_pitch_joint: limit lower=-1.3962634015954636 upper=1.0471975511965976 effort=45 velocity=14.660765716752369 -> lower=-1.2217 upper=1.2217 effort=30 velocity=10
- joint R_ankle_pitch_joint: axis 0 0 -1 -> 0 0 1; limit lower=-1.3962634015954636 upper=1.0471975511965976 effort=45 velocity=14.660765716752369 -> lower=-1.2217 upper=1.2217 effort=30 velocity=10

Commit message: Auxilaris sind hinzugefügt

File: legged_gym/resources/robots/x02/urdf/x02.urdf (robot description, URDF)
Before this commit: robot X02Lite, 50 links, 49 joints
Joints:
- joint auxiliary_left_ankle_roll_joint1: origin xyz=0.035 0.1 0 rpy=0 0 0 -> xyz=0 0 0.1 rpy=0 0 0
- joint auxiliary_left_ankle_roll_joint2: origin xyz=0.035 -0.1 0 rpy=0 0 0 -> xyz=0 0 -0.1 rpy=0 0 0
- joint auxiliary_left_ankle_roll_joint3: origin xyz=0.2 0 0 rpy=0 0 0 -> xyz=0 -0.2 0 rpy=0 0 0
- joint auxiliary_left_ankle_roll_joint4: origin xyz=-0.15 0 0 rpy=0 0 0 -> xyz=0 0.15 0 rpy=0 0 0
- joint auxiliary_right_ankle_roll_joint1: origin xyz=0.035 0.1 0 rpy=0 0 0 -> xyz=0 0 0.1 rpy=0 0 0
- joint auxiliary_right_ankle_roll_joint2: origin xyz=0.035 -0.1 0 rpy=0 0 0 -> xyz=0 0 -0.1 rpy=0 0 0
- joint auxiliary_right_ankle_roll_joint3: origin xyz=0.2 0 0 rpy=0 0 0 -> xyz=0 -0.2 0 rpy=0 0 0
- joint auxiliary_right_ankle_roll_joint4: origin xyz=-0.15 0 0 rpy=0 0 0 -> xyz=0 0.15 0 rpy=0 0 0

Commit message: ankle point links gefixed

File: legged_gym/resources/robots/x02/urdf/x02.urdf (robot description, URDF)
Before this commit: robot X02Lite, 50 links, 49 joints
Joints:
- joint auxiliary_left_ankle_roll_joint3: origin xyz=0 -0.2 0 rpy=0 0 0 -> xyz=0 0.2 0 rpy=0 0 0
- joint auxiliary_left_ankle_roll_joint4: origin xyz=0 0.15 0 rpy=0 0 0 -> xyz=0 -0.15 0 rpy=0 0 0

Commit message: shoulder fixed and ankle keyframes

File: legged_gym/resources/robots/x02/urdf/x02.urdf (robot description, URDF)
Before this commit: robot X02Lite, 50 links, 49 joints
Links:
- added link keyframe_left_ankle_link
- added link keyframe_right_ankle_link
Joints:
- added joint keyframe_left_ankle_joint: type fixed, parent L_ankle_pitch_Link, child keyframe_left_ankle_link, origin xyz=0 0 0 rpy=0 0 0
- added joint keyframe_right_ankle_joint: type fixed, parent R_ankle_pitch_Link, child keyframe_right_ankle_link, origin xyz=0 0 0 rpy=0 0 0
- joint L_elbow_joint: limit lower=0.0 upper=2.5307274153917776 effort=14 velocity=5.235987755982989 -> lower=-1.57 upper=0.9 effort=24 velocity=5.235987755982989
- joint R_elbow_joint: limit lower=0 upper=1.5707963267949 effort=14 velocity=5.235987755982989 -> lower=-1.57 upper=0.9 effort=24 velocity=5.235987755982989

Commit message: hind,mid,front_link richtig hinzugefügt und training: arme_und_fußfetisch gestartet

File: legged_gym/resources/robots/x02/urdf/x02.urdf (robot description, URDF)
Before this commit: robot X02Lite, 52 links, 51 joints
Joints:
- joint left_foot_front_joint: origin xyz=0.18 0 -0.06 rpy=0 0 0 -> xyz=0.087 0.18 0 rpy=0 0 0
- joint left_foot_hind_joint: origin xyz=-0.09 0 -0.06 rpy=0 0 0 -> xyz=0.087 -0.09 0 rpy=0 0 0
- joint left_foot_mid_joint: origin xyz=0.0 0 -0.06 rpy=0 0 0 -> xyz=0.087 0 0 rpy=0 0 0
- joint right_foot_front_joint: origin xyz=0.18 0 -0.06 rpy=0 0 0 -> xyz=0.087 -0.18 0 rpy=0 0 0
- joint right_foot_hind_joint: origin xyz=-0.09 0 -0.06 rpy=0 0 0 -> xyz=0.087 0.09 0 rpy=0 0 0
- joint right_foot_mid_joint: origin xyz=0.0 0 -0.06 rpy=0 0 0 -> xyz=0.087 0 0 rpy=0 0 0

Commit message: Mass und limit Werte der x02.urdf und x2_2.urdf stimmen bis Zeile 400 überein, ab hier dann Torso/waist schlammassel

File: legged_gym/resources/robots/x02/urdf/x02.urdf (robot description, URDF)
Before this commit: robot X02Lite, 52 links, 51 joints
Links:
- link R_hip_yaw_Link: mass 0.907 -> 1.758
Joints:
- joint L_hip_pitch_joint: limit lower=-0.5235987755982988 upper=2.007128639793479 effort=72 velocity=9.16297857297023 -> lower=-0.5236 upper=2.0071 effort=72 velocity=9.163
- joint L_hip_roll_joint: limit lower=-0.2617993877991494 upper=0.7853981633974483 effort=50 velocity=10.471975511965978 -> lower=-0.2618 upper=0.7854 effort=50 velocity=10.471975511965978
- joint L_hip_yaw_joint: limit lower=-0.7853981633974483 upper=0.7853981633974483 effort=50 velocity=10.471975511965978 -> lower=-0.7854 upper=0.7854 effort=50 velocity=10.472
- joint L_knee_pitch_joint: limit lower=-2.443460952792061 upper=0.08726646259971647 effort=150 velocity=7.3303828583761845 -> lower=-2.4435 upper=0.0873 effort=150 velocity=7.3303828583761845
- joint R_hip_pitch_joint: limit lower=-0.5235987755982988 upper=2.007128639793479 effort=72 velocity=9.16297857297023 -> lower=-0.5236 upper=2.0071 effort=72 velocity=9.163
- joint R_hip_roll_joint: limit lower=-0.2617993877991494 upper=0.7853981633974483 effort=50 velocity=10.471975511965978 -> lower=-0.2618 upper=0.7854 effort=50 velocity=10.472
- joint R_hip_yaw_joint: limit lower=-0.7853981633974483 upper=0.7853981633974483 effort=50 velocity=10.471975511965978 -> lower=-0.7854 upper=0.7854 effort=50 velocity=10.472
- joint R_knee_pitch_joint: limit lower=-2.443460952792061 upper=0.08726646259971647 effort=150 velocity=7.3303828583761845 -> lower=-2.4435 upper=0.0873 effort=150 velocity=7.3304

Commit message: x2_2 URDF wurde um pelvis, und hip_yaw aus x02 erweitert, Waist ist raus, außerdem sind bis hip_roll alle joints der beide soweit richtig

File: legged_gym/resources/robots/x02/urdf/x02.urdf (robot description, URDF)
Before this commit: robot X02Lite, 52 links, 51 joints
Links:
- link R_hip_yaw_Link: mass 1.758 -> 0.907

File: legged_gym/resources/robots/x02_2/x2_2.urdf (robot description, URDF)
Before this commit: robot x2, 23 links, 22 joints
Links:
- removed link waist_yaw_link
- link L_hip_yaw_link: geometry collision mesh filename=../meshes/L_hip_yaw_link.STL; visual mesh filename=../meshes/L_hip_yaw_link.STL
- link R_hip_yaw_link: mass 1.758 -> 0.907; geometry collision mesh filename=../meshes/R_hip_yaw_link.STL; visual mesh filename=../meshes/R_hip_yaw_link.STL
- link pelvis_link: geometry collision mesh filename=../meshes/pelvis_link.STL; visual mesh filename=../meshes/pelvis_link.STL
Joints:
- removed joint waist_yaw
- joint L_hip_roll: origin xyz=-0.0095 0.1 0 rpy=0 0 0 -> xyz=-0.0095 0.1 -0.0474 rpy=0 0 0
- joint L_hip_yaw: origin xyz=0 0 0 rpy=0 0 0 -> xyz=0 0 -0.06 rpy=0 0 0
- joint R_hip_yaw: origin xyz=0 0 0 rpy=0 0 0 -> xyz=0 0 -0.1074 rpy=0 0 0
- joint torso_joint: axis 0 0 0 -> 0 0 1; limit (none) -> lower=-0.785 upper=0.785 effort=50 velocity=10.471975511965978; origin xyz=0 0 0.03675 rpy=0 0 0 -> xyz=0 0 0 rpy=0 0 0; parent waist_yaw_link -> pelvis_link

Commit message: alle Gewichte und Limits stimmen jetzt in der x2_2.urdf

File: legged_gym/resources/robots/x02/urdf/x02.urdf (robot description, URDF)
Before this commit: robot X02Lite, 52 links, 51 joints
Joints:
- joint L_shoulder_yaw_joint: limit lower=-2.2689280275926285 upper=2.2689280275926285 effort=14 velocity=5.235987755982989 -> lower=-0.66 upper=1 effort=14 velocity=5.235987755982989
- joint R_shoulder_yaw_joint: limit lower=-2.2689280275926285 upper=2.2689280275926285 effort=14 velocity=5.235987755982989 -> lower=-0.66 upper=1 effort=14 velocity=5.235987755982989

File: legged_gym/resources/robots/x02_2/x2_2.urdf (robot description, URDF)
Before this commit: robot x2, 22 links, 21 joints
Links:
- removed link L_elbow_pitch_link
- removed link R_elbow_pitch_link
- added link L_elbow_link, mass 0.24; collision mesh filename=meshes/L_elbow_pitch_link.STL; visual mesh filename=meshes/L_elbow_pitch_link.STL
- added link R_elbow_link, mass 0.24; collision mesh filename=meshes/R_elbow_pitch_link.STL; visual mesh filename=meshes/R_elbow_pitch_link.STL
- link L_shoulder_pitch_link: mass 0.08 -> 0.3
- link L_shoulder_roll_link: mass 0.8 -> 0.704
- link L_shoulder_yaw_link: mass 0.5 -> 0.523
- link R_shoulder_pitch_link: mass 0.08 -> 0.3
- link R_shoulder_roll_link: mass 0.8 -> 0.704
- link R_shoulder_yaw_link: mass 0.5 -> 0.523
- link head_link: mass 1.67 -> 1.177
- link torso_link: mass 0.0051207 -> 9.2618
Joints:
- removed joint L_elbow_pitch_joint
- removed joint R_elbow_pitch_joint
- added joint L_elbow_joint: type revolute, parent L_shoulder_yaw_link, child L_elbow_link, origin xyz=0.01 0 -0.173 rpy=0 -1.57 0, axis 0 -1 0, limit lower=-1.57 upper=0.9 effort=24 velocity=5.236
- added joint R_elbow_joint: type revolute, parent R_shoulder_yaw_link, child R_elbow_link, origin xyz=0.010039 0 -0.173 rpy=0 -1.57 0, axis 0 -1 0, limit lower=-1.57 upper=0.9 effort=24 velocity=5.236
- joint L_shoulder_pitch_joint: limit lower=-1.57 upper=3.14 effort=66 velocity=30 -> lower=-1.57 upper=3.14 effort=18 velocity=5.236
- joint L_shoulder_roll_joint: limit lower=-0.35 upper=1.57 effort=66 velocity=30 -> lower=0 upper=3.141 effort=14 velocity=5.236
- joint L_shoulder_yaw_joint: limit lower=-2.618 upper=2.618 effort=45 velocity=30 -> lower=-0.66 upper=1 effort=14 velocity=5.236
- joint R_shoulder_pitch_joint: limit lower=-1.57 upper=3.14 effort=66 velocity=30 -> lower=-1.57 upper=3.14 effort=18 velocity=5.236
- joint R_shoulder_roll_joint: limit lower=-0.35 upper=1.57 effort=66 velocity=30 -> lower=0 upper=3.141 effort=14 velocity=5.236
- joint R_shoulder_yaw_joint: limit lower=-2.618 upper=2.618 effort=45 velocity=30 -> lower=-0.66 upper=1 effort=14 velocity=5.236
