Commit message: all joint positions correct

File: legged_gym/resources/robots/x02_2/x2_2.urdf (robot description, URDF)
Before this commit: robot x2, 22 links, 21 joints
Joints:
- joint L_hip_pitch: origin xyz=0.0085 -0.00100000000000001 -0.11 rpy=0 0 0 -> xyz=0.0085 0 -0.11 rpy=0 0 0
- joint R_hip_pitch: origin xyz=0.0085 -0.001 -0.11 rpy=0 0 0 -> xyz=0.0085 0 -0.11 rpy=0 0 0

Commit message: x2_2 URDF cleaned and Joint names changed

File: legged_gym/resources/robots/x02_2/x2_2.urdf (robot description, URDF)
Before this commit: robot x2, 22 links, 21 joints
Links:
- link L_hip_roll_link: geometry collision mesh filename=meshes/L_hip_roll_link.STL; visual mesh filename=meshes/L_hip_roll_link.STL
- link R_hip_roll_link: geometry collision mesh filename=meshes/R_hip_roll_link.STL; visual mesh filename=meshes/R_hip_roll_link.STL
Joints:
- removed joint L_ankle_pitch
- removed joint L_elbow_pitch
- removed joint L_hip_pitch
- removed joint L_hip_roll
- removed joint L_hip_yaw
- removed joint L_knee_pitch
- removed joint L_shoulder_pitch
- removed joint L_shoulder_roll
- removed joint L_shoulder_yaw
- removed joint R_ankle_pitch
- removed joint R_elbow_pitch
- removed joint R_hip_pitch
- removed joint R_hip_roll
- removed joint R_hip_yaw
- removed joint R_knee_pitch
- removed joint R_shoulder_pitch
- removed joint R_shoulder_roll
- removed joint R_shoulder_yaw
- removed joint head
- removed joint logo
- added joint L_ankle_pitch_joint: type revolute, parent L_knee_pitch_link, child L_ankle_pitch_link, origin xyz=0 0 -0.35 rpy=0 0 0, axis 0 -1 0, limit lower=-1.2217 upper=1.2217 effort=30 velocity=10
- added joint L_elbow_pitch_joint: type revolute, parent L_shoulder_yaw_link, child L_elbow_pitch_link, origin xyz=0.01 0 -0.173 rpy=0 -1.57 0, axis 0 -1 0, limit lower=-2.443 upper=2.443 effort=83.5 velocity=43
- added joint L_hip_pitch_joint: type revolute, parent L_hip_roll_link, child L_hip_pitch_link, origin xyz=0.0085 0 -0.11 rpy=0 0 0, axis 0 -1 0, limit lower=-0.5236 upper=2.0071 effort=72 velocity=9.163
- added joint L_hip_roll_joint: type revolute, parent L_hip_yaw_link, child L_hip_roll_link, origin xyz=-0.0095 0.1 -0.0474 rpy=0 0 0, axis 1 0 0, limit lower=-0.2618 upper=0.7854 effort=50 velocity=10.471975511965978
- added joint L_hip_yaw_joint: type revolute, parent pelvis_link, child L_hip_yaw_link, origin xyz=0 0 -0.06 rpy=0 0 0, axis 0 0 1, limit lower=-0.7854 upper=0.7854 effort=50 velocity=10.472
- added joint L_knee_pitch_joint: type revolute, parent L_hip_pitch_link, child L_knee_pitch_link, origin xyz=0 0 -0.35 rpy=0 0 0, axis 0 -1 0, limit lower=-2.4435 upper=0.0873 effort=60 velocity=7.3304
- added joint L_shoulder_pitch_joint: type revolute, parent torso_link, child L_shoulder_pitch_link, origin xyz=-0.01 0.14477 0.31534 rpy=0.17453 0 0, axis 0 -1 0, limit lower=-1.57 upper=3.14 effort=66 velocity=30
- added joint L_shoulder_roll_joint: type revolute, parent L_shoulder_pitch_link, child L_shoulder_roll_link, origin xyz=0 0.061 0 rpy=-0.17453 0 0, axis 1 0 0, limit lower=-0.35 upper=1.57 effort=66 velocity=30
- added joint L_shoulder_yaw_joint: type revolute, parent L_shoulder_roll_link, child L_shoulder_yaw_link, origin xyz=0 0 -0.112 rpy=0 0 0, axis 0 0 1, limit lower=-2.618 upper=2.618 effort=45 velocity=30
- added joint R_ankle_pitch_joint: type revolute, parent R_knee_pitch_link, child R_ankle_pitch_link, origin xyz=0 0 -0.35 rpy=0 0 0, axis 0 -1 0, limit lower=-1.2217 upper=1.2217 effort=30 velocity=10
- added joint R_elbow_pitch_joint: type revolute, parent R_shoulder_yaw_link, child R_elbow_pitch_link, origin xyz=0.010039 0 -0.173 rpy=0 -1.57 0, axis 0 -1 0, limit lower=-2.443 upper=2.443 effort=83.5 velocity=43
- added joint R_hip_pitch_joint: type revolute, parent R_hip_roll_link, child R_hip_pitch_link, origin xyz=0.0085 0 -0.11 rpy=0 0 0, axis 0 -1 0, limit lower=-0.5236 upper=2.0071 effort=72 velocity=9.163
- added joint R_hip_roll_joint: type revolute, parent R_hip_yaw_link, child R_hip_roll_link, origin xyz=-0.0095 -0.1 0 rpy=0 0 0, axis -1 0 0, limit lower=-0.2618 upper=0.7854 effort=50 velocity=10.472
- added joint R_hip_yaw_joint: type revolute, parent pelvis_link, child R_hip_yaw_link, origin xyz=0 0 -0.1074 rpy=0 0 0, axis 0 0 -1, limit lower=-0.7854 upper=0.7854 effort=50 velocity=10.472
- added joint R_knee_pitch_joint: type revolute, parent R_hip_pitch_link, child R_knee_pitch_link, origin xyz=0 0 -0.35 rpy=0 0 0, axis 0 -1 0, limit lower=-2.4435 upper=0.0873 effort=60 velocity=7.3304
- added joint R_shoulder_pitch_joint: type revolute, parent torso_link, child R_shoulder_pitch_link, origin xyz=-0.01 -0.14477 0.31534 rpy=-0.17453 0 0, axis 0 -1 0, limit lower=-1.57 upper=3.14 effort=66 velocity=30
- added joint R_shoulder_roll_joint: type revolute, parent R_shoulder_pitch_link, child R_shoulder_roll_link, origin xyz=0 -0.061 0 rpy=0.17453 0 0, axis -1 0 0, limit lower=-0.35 upper=1.57 effort=66 velocity=30
- added joint R_shoulder_yaw_joint: type revolute, parent R_shoulder_roll_link, child R_shoulder_yaw_link, origin xyz=-3.8964E-05 0 -0.112 rpy=0 0 0, axis 0 0 -1, limit lower=-2.618 upper=2.618 effort=45 velocity=30
- added joint head_joint: type fixed, parent torso_link, child head_link, origin xyz=0 0 0.3645 rpy=0 0 0, axis 0 0 1, limit lower=-1.571 upper=1.571 effort=50 velocity=5
- added joint logo_joint: type fixed, parent torso_link, child logo_link, origin xyz=0 0 0 rpy=0 0 0, axis 0 0 0

Commit message: urdf hat Keyframes, Auxiliaryties und foot_links

File: legged_gym/resources/robots/x02_2/x2_2.urdf (robot description, URDF)
Before this commit: robot x2, 22 links, 21 joints
Links:
- added link auxiliary_left_ankle_roll_link1; visual sphere radius=0.01
- added link auxiliary_left_ankle_roll_link2; visual sphere radius=0.01
- added link auxiliary_left_ankle_roll_link3; visual sphere radius=0.01
- added link auxiliary_left_ankle_roll_link4; visual sphere radius=0.01
- added link auxiliary_right_ankle_roll_link1; visual sphere radius=0.01
- added link auxiliary_right_ankle_roll_link2; visual sphere radius=0.01
- added link auxiliary_right_ankle_roll_link3; visual sphere radius=0.01
- added link auxiliary_right_ankle_roll_link4; visual sphere radius=0.01
- added link keyframe_head_link
- added link keyframe_left_ankle_link
- added link keyframe_left_collar_link
- added link keyframe_left_elbow_link
- added link keyframe_left_hip_link
- added link keyframe_left_knee_link
- added link keyframe_left_shoulder_link
- added link keyframe_pelvis_link
- added link keyframe_right_ankle_link
- added link keyframe_right_collar_link
- added link keyframe_right_elbow_link
- added link keyframe_right_hip_link
- added link keyframe_right_knee_link
- added link keyframe_right_shoulder_link
- added link keyframe_torso_link
- added link left_foot_front_link
- added link left_foot_hind_link
- added link left_foot_mid_link
- added link right_foot_front_link
- added link right_foot_hind_link
- added link right_foot_mid_link
Joints:
- added joint auxiliary_left_ankle_roll_joint1: type fixed, parent L_ankle_pitch_link, child auxiliary_left_ankle_roll_link1, origin xyz=0.035 0.1 0 rpy=0 0 0
- added joint auxiliary_left_ankle_roll_joint2: type fixed, parent L_ankle_pitch_link, child auxiliary_left_ankle_roll_link2, origin xyz=0.035 -0.1 0 rpy=0 0 0
- added joint auxiliary_left_ankle_roll_joint3: type fixed, parent L_ankle_pitch_link, child auxiliary_left_ankle_roll_link3, origin xyz=0.2 0 0 rpy=0 0 0
- added joint auxiliary_left_ankle_roll_joint4: type fixed, parent L_ankle_pitch_link, child auxiliary_left_ankle_roll_link4, origin xyz=-0.15 0 0 rpy=0 0 0
- added joint auxiliary_right_ankle_roll_joint1: type fixed, parent R_ankle_pitch_link, child auxiliary_right_ankle_roll_link1, origin xyz=0.035 0.1 0 rpy=0 0 0
- added joint auxiliary_right_ankle_roll_joint2: type fixed, parent R_ankle_pitch_link, child auxiliary_right_ankle_roll_link2, origin xyz=0.035 -0.1 0 rpy=0 0 0
- added joint auxiliary_right_ankle_roll_joint3: type fixed, parent R_ankle_pitch_link, child auxiliary_right_ankle_roll_link3, origin xyz=0.2 0 0 rpy=0 0 0
- added joint auxiliary_right_ankle_roll_joint4: type fixed, parent R_ankle_pitch_link, child auxiliary_right_ankle_roll_link4, origin xyz=-0.15 0 0 rpy=0 0 0
- added joint keyframe_head_joint: type fixed, parent torso_link, child keyframe_head_link, origin xyz=0 0 0.45 rpy=0 0 0
- added joint keyframe_left_ankle_joint: type fixed, parent L_ankle_pitch_link, child keyframe_left_ankle_link, origin xyz=0 0 0 rpy=0 0 0
- added joint keyframe_left_collar_joint: type fixed, parent L_shoulder_pitch_link, child keyframe_left_collar_link, origin xyz=0 0 0.02 rpy=0 0 0
- added joint keyframe_left_elbow_joint: type fixed, parent L_elbow_link, child keyframe_left_elbow_link, origin xyz=0 0 0 rpy=0 0 0
- added joint keyframe_left_hip_joint: type fixed, parent L_hip_roll_link, child keyframe_left_hip_link, origin xyz=0 0 0 rpy=0 0 0
- added joint keyframe_left_knee_joint: type fixed, parent L_knee_pitch_link, child keyframe_left_knee_link, origin xyz=0 0 0 rpy=0 0 0
- added joint keyframe_left_shoulder_joint: type fixed, parent L_shoulder_roll_link, child keyframe_left_shoulder_link, origin xyz=0 0 0 rpy=0 0 0
- added joint keyframe_pelvis_joint: type fixed, parent pelvis_link, child keyframe_pelvis_link, origin xyz=0 0 -0.075 rpy=0 0 0
- added joint keyframe_right_ankle_joint: type fixed, parent R_ankle_pitch_link, child keyframe_right_ankle_link, origin xyz=0 0 0 rpy=0 0 0
- added joint keyframe_right_collar_joint: type fixed, parent R_shoulder_pitch_link, child keyframe_right_collar_link, origin xyz=0 0 0.02 rpy=0 0 0
- added joint keyframe_right_elbow_joint: type fixed, parent R_elbow_link, child keyframe_right_elbow_link, origin xyz=0 0 0 rpy=0 0 0
- added joint keyframe_right_hip_joint: type fixed, parent R_hip_roll_link, child keyframe_right_hip_link, origin xyz=0 0 0 rpy=0 0 0
- added joint keyframe_right_knee_joint: type fixed, parent R_knee_pitch_link, child keyframe_right_knee_link, origin xyz=0 0 0 rpy=0 0 0
- added joint keyframe_right_shoulder_joint: type fixed, parent R_shoulder_roll_link, child keyframe_right_shoulder_link, origin xyz=0 0 0 rpy=0 0 0
- added joint keyframe_torso_joint: type fixed, parent torso_link, child keyframe_torso_link, origin xyz=0 0 0.2 rpy=0 0 0
- added joint left_foot_front_joint: type fixed, parent L_ankle_pitch_link, child left_foot_front_link, origin xyz=0.15 0 -0.087 rpy=0 0 0
- added joint left_foot_hind_joint: type fixed, parent L_ankle_pitch_link, child left_foot_hind_link, origin xyz=-0.095 0 -0.087 rpy=0 0 0
- added joint left_foot_mid_joint: type fixed, parent L_ankle_pitch_link, child left_foot_mid_link, origin xyz=0.0 0 -0.087 rpy=0 0 0
- added joint right_foot_front_joint: type fixed, parent R_ankle_pitch_link, child right_foot_front_link, origin xyz=0.15 0 -0.087 rpy=0 0 0
- added joint right_foot_hind_joint: type fixed, parent R_ankle_pitch_link, child right_foot_hind_link, origin xyz=-0.095 0 -0.087 rpy=0 0 0
- added joint right_foot_mid_joint: type fixed, parent R_ankle_pitch_link, child right_foot_mid_link, origin xyz=0.0 0 -0.087 rpy=0 0 0

Commit message: refactoring in der Urdf, inshallah jetzt ground parallel reward

File: legged_gym/resources/robots/x02_2/x2_2.urdf (robot description, URDF)
Before this commit: robot x2, 51 links, 50 joints
Links:
- removed link L_ankle_pitch_link
- removed link L_elbow_link
- removed link L_hip_pitch_link
- removed link L_hip_roll_link
- removed link L_hip_yaw_link
- removed link L_knee_pitch_link
- removed link L_shoulder_pitch_link
- removed link L_shoulder_roll_link
- removed link L_shoulder_yaw_link
- removed link R_ankle_pitch_link
- removed link R_elbow_link
- removed link R_hip_pitch_link
- removed link R_hip_roll_link
- removed link R_hip_yaw_link
- removed link R_knee_pitch_link
- removed link R_shoulder_pitch_link
- removed link R_shoulder_roll_link
- removed link R_shoulder_yaw_link
- added link left_ankle_pitch_link, mass 0.556154115746433; collision sphere radius=0.005; collision sphere radius=0.005
- added link left_elbow_link, mass 0.24; collision mesh filename=meshes/L_elbow_pitch_link.STL; visual mesh filename=meshes/L_elbow_pitch_link.STL
- added link left_hip_pitch_link, mass 1.332; collision mesh filename=meshes/L_hip_pitch_link.STL; visual mesh filename=meshes/L_hip_pitch_link.STL
- added link left_hip_roll_link, mass 1.562; collision mesh filename=meshes/L_hip_roll_link.STL; visual mesh filename=meshes/L_hip_roll_link.STL
- added link left_hip_yaw_link, mass 1.758; collision mesh filename=meshes/L_hip_yaw_link.STL; visual mesh filename=meshes/L_hip_yaw_link.STL
- added link left_knee_pitch_link, mass 0.847; collision mesh filename=meshes/L_knee_pitch_link.STL; visual mesh filename=meshes/L_knee_pitch_link.STL
- added link left_shoulder_pitch_link, mass 0.3; collision mesh filename=meshes/L_shoulder_pitch_link.STL; visual mesh filename=meshes/L_shoulder_pitch_link.STL
- added link left_shoulder_roll_link, mass 0.704; collision mesh filename=meshes/L_shoulder_roll_link.STL; visual mesh filename=meshes/L_shoulder_roll_link.STL
- added link left_shoulder_yaw_link, mass 0.523; collision mesh filename=meshes/L_shoulder_yaw_link.STL; visual mesh filename=meshes/L_shoulder_yaw_link.STL
- added link right_ankle_pitch_link, mass 0.556160945494453; collision sphere radius=0.005; collision sphere radius=0.005
- added link right_elbow_link, mass 0.24; collision mesh filename=meshes/R_elbow_pitch_link.STL; visual mesh filename=meshes/R_elbow_pitch_link.STL
- added link right_hip_pitch_link, mass 1.332; collision mesh filename=meshes/R_hip_pitch_link.STL; visual mesh filename=meshes/R_hip_pitch_link.STL
- added link right_hip_roll_link, mass 1.562; collision mesh filename=meshes/R_hip_roll_link.STL; visual mesh filename=meshes/R_hip_roll_link.STL
- added link right_hip_yaw_link, mass 0.907; collision mesh filename=meshes/R_hip_yaw_link.STL; visual mesh filename=meshes/R_hip_yaw_link.STL
- added link right_knee_pitch_link, mass 0.847; collision mesh filename=meshes/R_knee_pitch_link.STL; visual mesh filename=meshes/R_knee_pitch_link.STL
- added link right_shoulder_pitch_link, mass 0.3; collision mesh filename=meshes/R_shoulder_pitch_link.STL; visual mesh filename=meshes/R_shoulder_pitch_link.STL
- added link right_shoulder_roll_link, mass 0.704; collision mesh filename=meshes/R_shoulder_roll_link.STL; visual mesh filename=meshes/R_shoulder_roll_link.STL
- added link right_shoulder_yaw_link, mass 0.523; collision mesh filename=meshes/R_shoulder_yaw_link.STL; visual mesh filename=meshes/R_shoulder_yaw_link.STL
- link pelvis_link: geometry collision mesh filename=meshes/pelvis_link.STL; visual mesh filename=meshes/pelvis_link.STL
Joints:
- removed joint L_ankle_pitch_joint
- removed joint L_elbow_joint
- removed joint L_hip_pitch_joint
- removed joint L_hip_roll_joint
- removed joint L_hip_yaw_joint
- removed joint L_knee_pitch_joint
- removed joint L_shoulder_pitch_joint
- removed joint L_shoulder_roll_joint
- removed joint L_shoulder_yaw_joint
- removed joint R_ankle_pitch_joint
- removed joint R_elbow_joint
- removed joint R_hip_pitch_joint
- removed joint R_hip_roll_joint
- removed joint R_hip_yaw_joint
- removed joint R_knee_pitch_joint
- removed joint R_shoulder_pitch_joint
- removed joint R_shoulder_roll_joint
- removed joint R_shoulder_yaw_joint
- added joint left_ankle_pitch_joint: type revolute, parent left_knee_pitch_link, child left_ankle_pitch_link, origin xyz=0 0 -0.35 rpy=0 0 0, axis 0 -1 0, limit lower=-1.2217 upper=1.2217 effort=30 velocity=10
- added joint left_elbow_joint: type revolute, parent left_shoulder_yaw_link, child left_elbow_link, origin xyz=0.01 0 -0.173 rpy=0 -1.57 0, axis 0 -1 0, limit lower=-1.57 upper=0.9 effort=24 velocity=5.236
- added joint left_hip_pitch_joint: type revolute, parent left_hip_roll_link, child left_hip_pitch_link, origin xyz=0.0085 0 -0.11 rpy=0 0 0, axis 0 -1 0, limit lower=-0.5236 upper=2.0071 effort=72 velocity=9.163
- added joint left_hip_roll_joint: type revolute, parent left_hip_yaw_link, child left_hip_roll_link, origin xyz=-0.0095 0.1 -0.0474 rpy=0 0 0, axis 1 0 0, limit lower=-0.2618 upper=0.7854 effort=50 velocity=10.471975511965978
- added joint left_hip_yaw_joint: type revolute, parent pelvis_link, child left_hip_yaw_link, origin xyz=0 0 -0.06 rpy=0 0 0, axis 0 0 1, limit lower=-0.7854 upper=0.7854 effort=50 velocity=10.472
- added joint left_knee_pitch_joint: type revolute, parent left_hip_pitch_link, child left_knee_pitch_link, origin xyz=0 0 -0.35 rpy=0 0 0, axis 0 -1 0, limit lower=-2.4435 upper=0.0873 effort=60 velocity=7.3304
- added joint left_shoulder_pitch_joint: type revolute, parent torso_link, child left_shoulder_pitch_link, origin xyz=-0.01 0.14477 0.31534 rpy=0.17453 0 0, axis 0 -1 0, limit lower=-1.57 upper=3.14 effort=18 velocity=5.236
- added joint left_shoulder_roll_joint: type revolute, parent left_shoulder_pitch_link, child left_shoulder_roll_link, origin xyz=0 0.061 0 rpy=-0.17453 0 0, axis 1 0 0, limit lower=0 upper=3.141 effort=14 velocity=5.236
- added joint left_shoulder_yaw_joint: type revolute, parent left_shoulder_roll_link, child left_shoulder_yaw_link, origin xyz=0 0 -0.112 rpy=0 0 0, axis 0 0 1, limit lower=-0.66 upper=1 effort=14 velocity=5.236
- added joint right_ankle_pitch_joint: type revolute, parent right_knee_pitch_link, child right_ankle_pitch_link, origin xyz=0 0 -0.35 rpy=0 0 0, axis 0 -1 0, limit lower=-1.2217 upper=1.2217 effort=30 velocity=10
- added joint right_elbow_joint: type revolute, parent right_shoulder_yaw_link, child right_elbow_link, origin xyz=0.010039 0 -0.173 rpy=0 -1.57 0, axis 0 -1 0, limit lower=-1.57 upper=0.9 effort=24 velocity=5.236
- added joint right_hip_pitch_joint: type revolute, parent right_hip_roll_link, child right_hip_pitch_link, origin xyz=0.0085 0 -0.11 rpy=0 0 0, axis 0 -1 0, limit lower=-0.5236 upper=2.0071 effort=72 velocity=9.163
- added joint right_hip_roll_joint: type revolute, parent right_hip_yaw_link, child right_hip_roll_link, origin xyz=-0.0095 -0.1 0 rpy=0 0 0, axis -1 0 0, limit lower=-0.2618 upper=0.7854 effort=50 velocity=10.472
- added joint right_hip_yaw_joint: type revolute, parent pelvis_link, child right_hip_yaw_link, origin xyz=0 0 -0.1074 rpy=0 0 0, axis 0 0 -1, limit lower=-0.7854 upper=0.7854 effort=50 velocity=10.472
- added joint right_knee_pitch_joint: type revolute, parent right_hip_pitch_link, child right_knee_pitch_link, origin xyz=0 0 -0.35 rpy=0 0 0, axis 0 -1 0, limit lower=-2.4435 upper=0.0873 effort=60 velocity=7.3304
- added joint right_shoulder_pitch_joint: type revolute, parent torso_link, child right_shoulder_pitch_link, origin xyz=-0.01 -0.14477 0.31534 rpy=-0.17453 0 0, axis 0 -1 0, limit lower=-1.57 upper=3.14 effort=18 velocity=5.236
- added joint right_shoulder_roll_joint: type revolute, parent right_shoulder_pitch_link, child right_shoulder_roll_link, origin xyz=0 -0.061 0 rpy=0.17453 0 0, axis -1 0 0, limit lower=0 upper=3.141 effort=14 velocity=5.236
- added joint right_shoulder_yaw_joint: type revolute, parent right_shoulder_roll_link, child right_shoulder_yaw_link, origin xyz=-3.8964E-05 0 -0.112 rpy=0 0 0, axis 0 0 -1, limit lower=-0.66 upper=1 effort=14 velocity=5.236
- joint auxiliary_left_ankle_roll_joint1: parent L_ankle_pitch_link -> left_ankle_pitch_link
- joint auxiliary_left_ankle_roll_joint2: parent L_ankle_pitch_link -> left_ankle_pitch_link
- joint auxiliary_left_ankle_roll_joint3: parent L_ankle_pitch_link -> left_ankle_pitch_link
- joint auxiliary_left_ankle_roll_joint4: parent L_ankle_pitch_link -> left_ankle_pitch_link
- joint auxiliary_right_ankle_roll_joint1: parent R_ankle_pitch_link -> right_ankle_pitch_link
- joint auxiliary_right_ankle_roll_joint2: parent R_ankle_pitch_link -> right_ankle_pitch_link
- joint auxiliary_right_ankle_roll_joint3: parent R_ankle_pitch_link -> right_ankle_pitch_link
- joint auxiliary_right_ankle_roll_joint4: parent R_ankle_pitch_link -> right_ankle_pitch_link
- joint keyframe_left_ankle_joint: parent L_ankle_pitch_link -> left_ankle_pitch_link
- joint keyframe_left_collar_joint: parent L_shoulder_pitch_link -> left_shoulder_pitch_link
- joint keyframe_left_elbow_joint: parent L_elbow_link -> left_elbow_link
- joint keyframe_left_hip_joint: parent L_hip_roll_link -> left_hip_roll_link
- joint keyframe_left_knee_joint: parent L_knee_pitch_link -> left_knee_pitch_link
- joint keyframe_left_shoulder_joint: parent L_shoulder_roll_link -> left_shoulder_roll_link
- joint keyframe_right_ankle_joint: parent R_ankle_pitch_link -> right_ankle_pitch_link
- joint keyframe_right_collar_joint: parent R_shoulder_pitch_link -> right_shoulder_pitch_link
- joint keyframe_right_elbow_joint: parent R_elbow_link -> right_elbow_link
- joint keyframe_right_hip_joint: parent R_hip_roll_link -> right_hip_roll_link
- joint keyframe_right_knee_joint: parent R_knee_pitch_link -> right_knee_pitch_link
- joint keyframe_right_shoulder_joint: parent R_shoulder_roll_link -> right_shoulder_roll_link
- joint left_foot_front_joint: parent L_ankle_pitch_link -> left_ankle_pitch_link
- joint left_foot_hind_joint: parent L_ankle_pitch_link -> left_ankle_pitch_link
- joint left_foot_mid_joint: parent L_ankle_pitch_link -> left_ankle_pitch_link
- joint right_foot_front_joint: parent R_ankle_pitch_link -> right_ankle_pitch_link
- joint right_foot_hind_joint: parent R_ankle_pitch_link -> right_ankle_pitch_link
- joint right_foot_mid_joint: parent R_ankle_pitch_link -> right_ankle_pitch_link

Commit message: änderung in Start und ziel pose; stand training maybe_waist_deviation

File: legged_gym/resources/robots/x02_2/x2_2.urdf (robot description, URDF)
Before this commit: robot x2, 51 links, 50 joints
Joints:
- joint torso_joint: limit lower=-0.785 upper=0.785 effort=50 velocity=10.471975511965978 -> lower=-2.35 upper=2.35 effort=50 velocity=10.471975511965978
