Commit message: new hip_roll_link for X02

File: legged_gym/resources/robots/x02_2/x2_new_hip.urdf (robot description, URDF)
Before this commit: robot x2, 51 links, 50 joints
Links:
- link left_hip_roll_link: geometry collision mesh filename=meshes/L_hip_roll_Link_.STL; visual mesh filename=meshes/L_hip_roll_Link_.STL
- link right_hip_roll_link: geometry collision mesh filename=meshes/R_hip_roll_Link_.STL; visual mesh filename=meshes/R_hip_roll_Link_.STL
Joints:
- joint left_hip_pitch_joint: limit lower=-0.5236 upper=2.0071 effort=72 velocity=9.163 -> lower=-0.5235987755982988 upper=2.007128639793479 effort=72 velocity=9.16297857297023; origin xyz=0.0085 0 -0.11 rpy=0 0 0 -> xyz=0.092 -0.001 -2.97932823952292E-05 rpy=3.1416 1.5707963267949 0
- joint left_hip_roll_joint: axis 1 0 0 -> 0 0 -1; limit lower=-0.2618 upper=0.7854 effort=50 velocity=10.471975511965978 -> lower=-0.2617993877991494 upper=0.7853981633974483 effort=50 velocity=10.471975511965978; origin xyz=-0.0095 0.1 -0.0474 rpy=0 0 0 -> xyz=0 0.09 -0.0474 rpy=3.14159265358979 1.5707963267949 0
- joint right_hip_pitch_joint: limit lower=-0.5236 upper=2.0071 effort=72 velocity=9.163 -> lower=-0.5235987755982988 upper=2.007128639793479 effort=72 velocity=9.16297857297023; origin xyz=0.0085 0 -0.11 rpy=0 0 0 -> xyz=0.092 -0.00100000000000001 2.97932823952229E-05 rpy= 0 -1.5707963267949 0
- joint right_hip_roll_joint: axis -1 0 0 -> 0 0 -1; limit lower=-0.2618 upper=0.7854 effort=50 velocity=10.472 -> lower=-0.2617993877991494 upper=0.7853981633974483 effort=50 velocity=10.471975511965978; origin xyz=-0.0095 -0.1 0 rpy=0 0 0 -> xyz=0 -0.09 0 rpy=0 1.5707963267949 0

Commit message: stronger arms + no velocity limit; run name: training_strong

File: legged_gym/resources/robots/x02_2/x2_new_hip.urdf (robot description, URDF)
Before this commit: robot x2, 51 links, 50 joints
Joints:
- joint left_elbow_joint: limit lower=-1.57 upper=0.9 effort=24 velocity=5.236 -> lower=-1.57 upper=0.9 effort=24 velocity=37
- joint left_shoulder_pitch_joint: limit lower=-1.57 upper=3.14 effort=18 velocity=5.236 -> lower=-1.57 upper=3.14 effort=24 velocity=37
- joint left_shoulder_roll_joint: limit lower=0 upper=3.141 effort=14 velocity=5.236 -> lower=0 upper=3.141 effort=24 velocity=37
- joint left_shoulder_yaw_joint: limit lower=-0.66 upper=1 effort=14 velocity=5.236 -> lower=-0.66 upper=1 effort=24 velocity=37
- joint right_elbow_joint: limit lower=-1.57 upper=0.9 effort=24 velocity=5.236 -> lower=-1.57 upper=0.9 effort=24 velocity=37
- joint right_shoulder_pitch_joint: limit lower=-1.57 upper=3.14 effort=18 velocity=5.236 -> lower=-1.57 upper=3.14 effort=24 velocity=37
- joint right_shoulder_roll_joint: limit lower=0 upper=3.141 effort=14 velocity=5.236 -> lower=0 upper=3.141 effort=24 velocity=37
- joint right_shoulder_yaw_joint: limit lower=-0.66 upper=1 effort=14 velocity=5.236 -> lower=-0.66 upper=1 effort=24 velocity=37

Commit message: weniger Joint-Limits, bischen veränderte base_height werte, x02_training_loose

File: legged_gym/resources/robots/x02_2/x2_new_hip.urdf (robot description, URDF)
Before this commit: robot x2, 51 links, 50 joints
Joints:
- joint left_hip_pitch_joint: limit lower=-0.5235987755982988 upper=2.007128639793479 effort=72 velocity=9.16297857297023 -> lower=-0.5235987755982988 upper=2.307128639793479 effort=72 velocity=9.16297857297023
- joint left_hip_roll_joint: limit lower=-0.2617993877991494 upper=0.7853981633974483 effort=50 velocity=10.471975511965978 -> lower=-0.2617993877991494 upper=1.57 effort=50 velocity=10.471975511965978
- joint left_hip_yaw_joint: limit lower=-0.7854 upper=0.7854 effort=50 velocity=10.472 -> lower=-1.3 upper=1.3 effort=50 velocity=10.472
- joint left_shoulder_yaw_joint: limit lower=-0.66 upper=1 effort=24 velocity=37 -> lower=-1 upper=1 effort=24 velocity=37
- joint right_hip_pitch_joint: limit lower=-0.5235987755982988 upper=2.007128639793479 effort=72 velocity=9.16297857297023 -> lower=-0.5235987755982988 upper=2.307128639793479 effort=72 velocity=9.16297857297023
- joint right_hip_roll_joint: limit lower=-0.2617993877991494 upper=0.7853981633974483 effort=50 velocity=10.471975511965978 -> lower=-0.2617993877991494 upper=1.57 effort=50 velocity=10.471975511965978
- joint right_hip_yaw_joint: limit lower=-0.7854 upper=0.7854 effort=50 velocity=10.472 -> lower=-1.3 upper=1.3 effort=50 velocity=10.472
- joint right_shoulder_yaw_joint: limit lower=-0.66 upper=1 effort=24 velocity=37 -> lower=-1 upper=1 effort=24 velocity=37

Commit message: post_task wieder aus, einschränkung von hip_yaw, x02_training_in_ketten

File: legged_gym/resources/robots/x02_2/x2_new_hip.urdf (robot description, URDF)
Before this commit: robot x2, 51 links, 50 joints
Joints:
- joint left_hip_yaw_joint: limit lower=-1.3 upper=1.3 effort=50 velocity=10.472 -> lower=-1.3 upper=1 effort=50 velocity=10.472
- joint right_hip_yaw_joint: limit lower=-1.3 upper=1.3 effort=50 velocity=10.472 -> lower=-1.3 upper=1 effort=50 velocity=10.472

Commit message: kopfhöhe angepasst, x02_training_low_height

File: legged_gym/resources/robots/x02_2/x2_new_hip.urdf (robot description, URDF)
Before this commit: robot x2, 51 links, 50 joints
Joints:
- joint left_hip_yaw_joint: limit lower=-1.3 upper=1 effort=50 velocity=10.472 -> lower=-1.3 upper=1.3 effort=50 velocity=10.472
- joint right_hip_yaw_joint: limit lower=-1.3 upper=1 effort=50 velocity=10.472 -> lower=-1.3 upper=1.3 effort=50 velocity=10.472
