Commit message: urdf change hin zu dicken hip_roll linkd, Einschränkungen im pelvis und roll, x02_training_prone4

File: legged_gym/resources/robots/x02_2/x2.urdf (robot description, URDF)
Before this commit: robot x2, 51 links, 50 joints
Joints:
- joint left_elbow_joint: limit lower=-1.57 upper=0.9 effort=24 velocity=5.236 -> lower=-1.57 upper=0.9 effort=24 velocity=37
- joint left_shoulder_pitch_joint: limit lower=-1.57 upper=3.14 effort=18 velocity=5.236 -> lower=-1.57 upper=3.14 effort=24 velocity=37
- joint left_shoulder_roll_joint: limit lower=0 upper=3.141 effort=14 velocity=5.236 -> lower=0 upper=3.141 effort=24 velocity=37
- joint left_shoulder_yaw_joint: limit lower=-0.66 upper=1 effort=14 velocity=5.236 -> lower=-1 upper=1 effort=24 velocity=37
- joint right_elbow_joint: limit lower=-1.57 upper=0.9 effort=24 velocity=5.236 -> lower=-1.57 upper=0.9 effort=24 velocity=37
- joint right_shoulder_pitch_joint: limit lower=-1.57 upper=3.14 effort=18 velocity=5.236 -> lower=-1.57 upper=3.14 effort=24 velocity=37
- joint right_shoulder_roll_joint: limit lower=0 upper=3.141 effort=14 velocity=5.236 -> lower=0 upper=3.141 effort=24 velocity=37
- joint right_shoulder_yaw_joint: limit lower=-0.66 upper=1 effort=14 velocity=5.236 -> lower=-1 upper=1 effort=24 velocity=37
- joint torso_joint: limit lower=-2.35 upper=2.35 effort=50 velocity=10.471975511965978 -> lower=-1 upper=1 effort=50 velocity=10.471975511965978

File: legged_gym/resources/robots/x02_2/x2_new_hip.urdf (robot description, URDF)
Before this commit: robot x2, 51 links, 50 joints
Joints:
- joint torso_joint: limit lower=-2.35 upper=2.35 effort=50 velocity=10.471975511965978 -> lower=-1 upper=1 effort=50 velocity=10.471975511965978

Commit message: Urdf Limits stimmen jetzt

File: legged_gym/resources/robots/x02_2/x2.urdf (robot description, URDF)
Before this commit: robot x2, 51 links, 50 joints
Links:
- link head_link: mass 1.177 -> 1.67
- link left_hip_pitch_link: mass 1.332 -> 1.664
- link left_hip_roll_link: mass 1.562 -> 2.667
- link left_knee_pitch_link: mass 0.847 -> 1.125
- link right_hip_pitch_link: mass 1.332 -> 1.664
- link right_hip_roll_link: mass 1.562 -> 2.667
- link right_knee_pitch_link: mass 0.847 -> 1.125
Joints:
- joint left_ankle_pitch_joint: limit lower=-1.2217 upper=1.2217 effort=30 velocity=10 -> lower=-1 upper=1 effort=30 velocity=10
- joint left_hip_pitch_joint: limit lower=-0.5236 upper=2.0071 effort=72 velocity=9.163 -> lower=-0.5236 upper=2.13 effort=72 velocity=9.163
- joint left_hip_roll_joint: limit lower=-0.2618 upper=0.7854 effort=50 velocity=10.471975511965978 -> lower=-0.2618 upper=0.524 effort=50 velocity=10.471975511965978
- joint left_hip_yaw_joint: limit lower=-0.7854 upper=0.7854 effort=50 velocity=10.472 -> lower=-0.55 upper=0.55 effort=50 velocity=10.472
- joint left_knee_pitch_joint: limit lower=-2.4435 upper=0.0873 effort=60 velocity=7.3304 -> lower=-2.3 upper=0 effort=60 velocity=7.3304
- joint left_shoulder_yaw_joint: limit lower=-1 upper=1 effort=24 velocity=37 -> lower=-2.1 upper=2.1 effort=24 velocity=37
- joint right_ankle_pitch_joint: limit lower=-1.2217 upper=1.2217 effort=30 velocity=10 -> lower=-1 upper=1 effort=30 velocity=10
- joint right_hip_pitch_joint: limit lower=-0.5236 upper=2.0071 effort=72 velocity=9.163 -> lower=-0.5236 upper=2.13 effort=72 velocity=9.163
- joint right_hip_roll_joint: limit lower=-0.2618 upper=0.7854 effort=50 velocity=10.472 -> lower=-0.2618 upper=0.524 effort=50 velocity=10.472
- joint right_hip_yaw_joint: limit lower=-0.7854 upper=0.7854 effort=50 velocity=10.472 -> lower=-0.55 upper=0.55 effort=50 velocity=10.472
- joint right_knee_pitch_joint: limit lower=-2.4435 upper=0.0873 effort=60 velocity=7.3304 -> lower=-2.3 upper=0 effort=60 velocity=7.3304
- joint right_shoulder_yaw_joint: limit lower=-1 upper=1 effort=24 velocity=37 -> lower=-2.1 upper=2.1 effort=24 velocity=37
