Commit message: mesh pfade changed

File: legged_gym/resources/robots/pi_plus_22dof/pi_plus_22dof.urdf (robot description, URDF)
Before this commit: robot pi_plus_24dof, 47 links, 46 joints
Links:
- link base_link: geometry collision box size=0.035 0.035 0.074; collision box size=0.045 0.055 0.045
- link head_pitch_link: geometry collision mesh filename=meshes/head_pitch_link.STL; visual mesh filename=meshes/head_pitch_link.STL
- link head_yaw_link: geometry collision mesh filename=meshes/head_yaw_link.STL; visual mesh filename=meshes/head_yaw_link.STL
- link l_ankle_pitch_link: geometry collision box size=0.006 0.06 0.03; collision box size=0.006 0.06 0.03
- link l_ankle_roll_link: geometry collision mesh filename=meshes/ankle_roll_link_simplify.STL; visual mesh filename=meshes/l_ankle_roll_link.STL
- link l_calf_link: geometry collision box size=0.01 0.02 0.055; collision mesh filename=meshes/l_calf_link_2.STL
- link l_elbow_link: geometry collision mesh filename=meshes/l_elbow_link.STL; visual mesh filename=meshes/l_elbow_link.STL
- link l_hip_pitch_link: geometry collision mesh filename=meshes/l_hip_pitch_link.STL; visual mesh filename=meshes/l_hip_pitch_link.STL
- link l_hip_roll_link: geometry collision mesh filename=meshes/l_hip_roll_link.STL; visual mesh filename=meshes/l_hip_roll_link.STL
- link l_shoulder_pitch_link: geometry collision mesh filename=meshes/l_shoulder_pitch_link.STL; visual mesh filename=meshes/l_shoulder_pitch_link.STL
- link l_shoulder_roll_link: geometry collision mesh filename=meshes/l_shoulder_roll_link.STL; visual mesh filename=meshes/l_shoulder_roll_link.STL
- link l_thigh_link: geometry collision mesh filename=meshes/l_thigh_link.STL; visual mesh filename=meshes/l_thigh_link.STL
- link l_upper_arm_link: geometry collision mesh filename=meshes/l_upper_arm_link.STL; visual mesh filename=meshes/l_upper_arm_link.STL
- link l_wrist_link: geometry collision mesh filename=meshes/l_wrist_link.STL; visual mesh filename=meshes/l_wrist_link.STL
- link r_ankle_pitch_link: geometry collision box size=0.006 0.06 0.03; collision box size=0.006 0.06 0.03
- link r_ankle_roll_link: geometry collision mesh filename=meshes/ankle_roll_link_simplify.STL; visual mesh filename=meshes/r_ankle_roll_link.STL
- link r_calf_link: geometry collision box size=0.01 0.02 0.055; collision mesh filename=meshes/r_calf_link_1.STL
- link r_elbow_link: geometry collision mesh filename=meshes/r_elbow_link.STL; visual mesh filename=meshes/r_elbow_link.STL
- link r_hip_pitch_link: geometry collision mesh filename=meshes/r_hip_pitch_link.STL; visual mesh filename=meshes/r_hip_pitch_link.STL
- link r_hip_roll_link: geometry collision mesh filename=meshes/r_hip_roll_link.STL; visual mesh filename=meshes/r_hip_roll_link.STL
- link r_shoulder_pitch_link: geometry collision mesh filename=meshes/r_shoulder_pitch_link.STL; visual mesh filename=meshes/r_shoulder_pitch_link.STL
- link r_shoulder_roll_link: geometry collision mesh filename=meshes/r_shoulder_roll_link.STL; visual mesh filename=meshes/r_shoulder_roll_link.STL
- link r_thigh_link: geometry collision mesh filename=meshes/r_thigh_link.STL; visual mesh filename=meshes/r_thigh_link.STL
- link r_upper_arm_link: geometry collision mesh filename=meshes/r_upper_arm_link.STL; visual mesh filename=meshes/r_upper_arm_link.STL
- link r_wrist_link: geometry collision mesh filename=meshes/r_wrist_link.STL; visual mesh filename=meshes/r_wrist_link.STL

Commit message: update head_link

File: legged_gym/resources/robots/pi_plus_22dof/pi_plus_22dof.urdf (robot description, URDF)
Before this commit: robot pi_plus_24dof, 47 links, 46 joints
Joints:
- joint keyframe_head_joint: origin xyz=0 0 0.08 rpy=0 0 0 -> xyz=0 0 0.15 rpy=0 0 0

Commit message: Limit joints

File: legged_gym/resources/robots/pi_plus_22dof/pi_plus_22dof.urdf (robot description, URDF)
Before this commit: robot pi_plus_24dof, 47 links, 46 joints
Joints:
- joint l_ankle_pitch_joint: limit lower=-0.97 upper=0.92 effort=20 velocity=5.45 -> lower=-0.5 upper=0.92 effort=20 velocity=5.45
- joint l_calf_joint: limit lower=-2.49 upper=2.49 effort=20 velocity=5.45 -> lower=-0.05 upper=1.65 effort=20 velocity=5.45
- joint r_ankle_pitch_joint: limit lower=-0.97 upper=0.92 effort=20 velocity=5.45 -> lower=-0.5 upper=0.92 effort=20 velocity=5.45
- joint r_calf_joint: limit lower=-2.49 upper=2.49 effort=20 velocity=5.45 -> lower=-0.05 upper=1.65 effort=20 velocity=5.45

Commit message: Tune params and joint limit

File: legged_gym/resources/robots/pi_plus_22dof/pi_plus_22dof.urdf (robot description, URDF)
Before this commit: robot pi_plus_24dof, 47 links, 46 joints
Joints:
- joint head_pitch_joint: limit lower=-0.34 upper=1.57 effort=3 velocity=30.37 -> lower=-0.34 upper=0.9 effort=3 velocity=30.37
- joint head_yaw_joint: limit lower=-1.39 upper=1.39 effort=3 velocity=30.37 -> lower=-0.3 upper=0.3 effort=3 velocity=30.37
- joint l_calf_joint: limit lower=-0.05 upper=1.65 effort=20 velocity=5.45 -> lower=-0.05 upper=2.4 effort=20 velocity=5.45
- joint l_elbow_joint: limit lower=-1.91 upper=1.91 effort=10 velocity=15.91 -> lower=-1.91 upper=0.0 effort=10 velocity=15.91
- joint l_hip_pitch_joint: limit lower=-3.12 upper=2.94 effort=20 velocity=5.45 -> lower=-1.45 upper=1.45 effort=20 velocity=5.45
- joint l_hip_roll_joint: limit lower=-0.31 upper=3.14 effort=20 velocity=5.45 -> lower=-0.31 upper=1.2 effort=20 velocity=5.45
- joint l_thigh_joint: limit lower=-2.87 upper=2.87 effort=20 velocity=5.45 -> lower=-1.2 upper=0.6 effort=20 velocity=5.45
- joint r_calf_joint: limit lower=-0.05 upper=1.65 effort=20 velocity=5.45 -> lower=-0.05 upper=2.4 effort=20 velocity=5.45
- joint r_elbow_joint: limit lower=-1.91 upper=1.91 effort=10 velocity=15.91 -> lower=-1.91 upper=0.0 effort=10 velocity=15.91
- joint r_hip_pitch_joint: limit lower=-3.12 upper=2.94 effort=20 velocity=5.45 -> lower=-1.45 upper=1.45 effort=20 velocity=5.45
- joint r_hip_roll_joint: limit lower=-3.14 upper=0.31 effort=20 velocity=5.45 -> lower=-1.2 upper=0.31 effort=20 velocity=5.45
- joint r_thigh_joint: limit lower=-2.87 upper=2.87 effort=20 velocity=5.45 -> lower=-1.2 upper=1.2 effort=20 velocity=5.45
