Commit message: stiffness an damping values correkt

File: legged_gym/resources/robots/pi_plus_torso/pi_plus_torso.urdf (robot description, URDF)
Before this commit: robot PiPlus_S_12L8A0G2H0W, 49 links, 48 joints
Joints:
- joint head_pitch_joint: limit lower=-1.23 upper=1.01 effort=3 velocity=30.37 -> lower=-1.23 upper=1.01 effort=2.5 velocity=30.37
- joint head_yaw_joint: limit lower=-1.43 upper=1.43 effort=3 velocity=30.37 -> lower=-1.43 upper=1.43 effort=2.5 velocity=30.37
