Commit message: target position changed + nan/inf checks for prone position rewards

File: legged_gym/resources/robots/pi_plus_torso/pi_plus.urdf (robot description, URDF)
Before this commit: robot PiPlus_S_12L8A0G2H0W, 52 links, 51 joints
Joints:
- joint l_shoulder_roll_joint: limit lower=-0.13 upper=3.34 effort=10 velocity=15.91 -> lower=-3.34 upper=0.13 effort=10 velocity=15.91
