Commit message: actuator2: flat-foot threshold for supine, hard knee limits
Starting point for the actuator2 trainings. Actuator parameters are
unchanged from actuator1; this only addresses two style problems seen
in the actuator1 policies.

- Feet not flat on the ground during phase 1/2 of the supine get-up:
  _reward_ground_parallel in host_ground now uses the binary threshold
  (var < 0.05) from host_ground_prone instead of the linear ramp
  (1 - var/0.15). The prone runs keep the feet noticeably flatter with
  it. Threshold is ~18 deg of foot roll instead of ~33 deg. Note that
  style_ground_parallel is still 25 for supine vs 20 for prone, which
  is now the full step height rather than a scale factor.
- Knees hyperextending into a non-human direction: hard limits in
  pi_plus_correct_limits.urdf, r_calf lower -2.14 -> -0.1 and l_calf
  upper 2.14 -> 0.1 (axes are mirrored, so human bend is r_calf
  positive / l_calf negative). Only the two <limit> lines changed;
  armature, damping/friction and the arm limits stay as they are.
  Applies to supine and prone, both configs load this URDF.
  _reward_knee_deviation cannot do this job: its |q| > 0.5 clause
  fires on any bend past 28 deg, so it is on for the whole get-up and
  carries no direction information.

Co-Authored-By: Claude Opus 5 <noreply@anthropic.com>
Claude-Session: https://claude.ai/code/session_012bBNoRFS17fa7ixLvCqY9T

File: legged_gym/resources/robots/pi_plus_torso/pi_plus_correct_limits.urdf (robot description, URDF)
Before this commit: robot PiPlus_S_12L8A0G2H0W, 54 links, 53 joints
Joints:
- joint l_calf_joint: limit lower=-2.26 upper=2.14 effort=20 velocity=5.45 -> lower=-2.26 upper=0.1 effort=20 velocity=5.45
- joint r_calf_joint: limit lower=-2.14 upper=2.26 effort=20 velocity=5.45 -> lower=-0.1 upper=2.26 effort=20 velocity=5.45
