Commit message: actuator3: disabled hard limits in urdf, did not work in sim2sim transfer. new knee extrention penalty added

File: legged_gym/resources/robots/pi_plus_torso/pi_plus_correct_limits.urdf (robot description, URDF)
Before this commit: robot PiPlus_S_12L8A0G2H0W, 54 links, 53 joints
Joints:
- joint l_calf_joint: limit lower=-2.26 upper=0.1 effort=20 velocity=5.45 -> lower=-2.26 upper=2.14 effort=20 velocity=5.45
- joint r_calf_joint: limit lower=-0.1 upper=2.26 effort=20 velocity=5.45 -> lower=-2.14 upper=2.26 effort=20 velocity=5.45
